Commit message: bigfootbot_description added urdf

File: bigfoot_description/urdf/bigfootbot.urdf (robot description, URDF)
Before this commit: robot basic_mobile_bot, 5 links, 4 joints
Links:
- link base_link: geometry collision box size=${base_length} ${base_width} ${base_height}; visual mesh filename=package://bigfootbot_description/meshes/frame.stl
