Commit message: bigfootbot_description

File: bigfootbot_description/urdf/bigfootbot.urdf (robot description, URDF)
Before this commit: robot bigfootbot, 5 links, 4 joints
Links:
- removed link front_caster
- removed link gps_link
- removed link imu_link
- link base_link: geometry collision box size=${base_length} ${base_width} ${base_height}; visual mesh filename=package://bigfootbot_description/meshes/frame_with_covers_2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 scale=0.001 0.001 0.001
Joints:
- removed joint caster_joint
- removed joint gps_joint
- removed joint imu_joint

Commit message: robot description - urdf file update, new stl file for base_link

File: bigfootbot_description/urdf/bigfootbot.urdf (robot description, URDF)
Before this commit: robot bigfootbot, 2 links, 1 joints
Links:
- link base_link: geometry collision box size=${base_length} ${base_width} ${base_height}; visual mesh filename=package://bigfootbot_description/meshes/frame_with_covers_2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
