Commit message: added xacro files and launch files

File: bigfootbot_description/urdf/bfb_common_properties.urdf.xacro (robot description, xacro)
@@ -27,4 +27,4 @@
   <xacro:property name="wheel_xoff" value="0.275"/>
   <!-- Maximum torque which the wheels can produce, in Nm -->
-  <xacro:property name="wheel_torque" value="20" />
+  <xacro:property name="wheel_torque" value="100" />
 </robot>

File: bigfootbot_description/urdf/bigfootbot_NEW.urdf.xacro (robot description, xacro)
@@ -9,12 +9,14 @@
   <!-- Drive wheel -->
   <xacro:include filename="$(find bigfootbot_description)/urdf/mech/wheel.urdf.xacro"/>
-  <!-- IMU -->
+  <!-- IMU (includes Gazebo plugin for sensor) -->
   <xacro:include filename="$(find bigfootbot_description)/urdf/sensors/imu.urdf.xacro"/>
-  <!-- LiDAR -->
+  <!-- LiDAR (includes Gazebo plugin for sensor) -->
   <xacro:include filename="$(find bigfootbot_description)/urdf/sensors/lidar.urdf.xacro"/>
+  <!-- GPS (includes Gazebo plugin for sensor) -->
+  <xacro:include filename="$(find bigfootbot_description)/urdf/sensors/gps.urdf.xacro"/>
   <!-- Drive controller (Gazebo plugin) -->
   <xacro:include filename="$(find bigfootbot_description)/urdf/controllers/skid_steer.urdf.xacro"/>
   <!-- Joint state publisher (Gazebo plugin) -->
-  <!--xacro:include filename="$(find bigfootbot_description)/urdf/controllers/joint_state_publisher.urdf.xacro"/-->
+  <xacro:include filename="$(find bigfootbot_description)/urdf/controllers/joint_state_publisher.urdf.xacro"/>
   <!-- Add robot base -->
   <xacro:base
@@ -37,4 +39,6 @@
   <!-- Add LiDAR -->
   <xacro:lidar/>
+  <!-- Add GPS -->
+  <xacro:gps/>
   <!-- Add drive controller (Gazebo plugin) -->
   <xacro:diff_drive_controller
@@ -44,8 +48,8 @@
   />
   <!-- Add joint state publisher (Gazebo plugin) -->
-  <!--xacro:joint_state_publisher
+  <xacro:joint_state_publisher
     front_left_whl_joint="drivewhl_fl_joint" front_right_whl_joint="drivewhl_fr_joint"
     rear_left_whl_joint="drivewhl_rl_joint" rear_right_whl_joint="drivewhl_rr_joint"
-  /-->
+  />
   <!-- *********************** GPS SETUP **********************************  -->
   <!--joint name="gps_joint" type="fixed">

File: bigfootbot_description/urdf/controllers/joint_state_publisher.urdf.xacro (robot description, xacro)
@@ -16,5 +16,5 @@
         <joint_name>drivewhl_fr_joint</joint_name>
         <joint_name>drivewhl_rl_joint</joint_name>
-        <joint_name>drivewhl_rr_joint</joint_name--
+        <joint_name>drivewhl_rr_joint</joint_name-->
       </plugin>
     </gazebo>

File: bigfootbot_description/urdf/mech/wheel.urdf.xacro (robot description, xacro)
@@ -25,8 +25,8 @@
     </link>
     <gazebo reference="${prefix}_link">
-      <mu1>0.7</mu1> <!-- friction coefficients for the two principle contact directions -->
-      <mu2>1.0</mu2> <!-- the static friction coefficient and the kinetic friction coefficient.-->
-      <!--kp>300000.0</kp--> <!-- contact stiffness -->
-      <!--kd></kd--> <!-- contact damping -->
+      <mu1>10</mu1> <!-- friction coefficients for the two principle contact directions -->
+      <mu2>7</mu2> <!-- the static friction coefficient and the kinetic (sliding) friction coefficient.-->
+      <!--kp>300000</kp--> <!-- contact stiffness -->
+      <!--kd>100</kd--> <!-- contact damping -->
       <!--material>Gazebo/Black</material-->
       <visual>
