Commit message: robot urdf files

File: bigfootbot_description/urdf/bigfootbot_NEW.urdf.xacro (robot description, xacro)
@@ -4,5 +4,5 @@
   <xacro:include filename="$(find bigfootbot_description)/urdf/bfb_common_properties.urdf.xacro"/>
   <!-- Inertial -->
-  <xacro:include filename="$(find bigfootbot_description)/urdf/inertials.urdf.xacro"/>
+  <!--xacro:include filename="$(find bigfootbot_description)/urdf/inertials.urdf.xacro"/-->
   <!-- Base -->
   <xacro:include filename="$(find bigfootbot_description)/urdf/mech/base.urdf.xacro"/>

File: bigfootbot_description/urdf/mech/base.urdf.xacro (robot description, xacro)
@@ -1,5 +1,7 @@
 <?xml version="1.0"?>
 <robot xmlns:xacro="http://ros.org/wiki/xacro">
-<!-- ********************** ROBOT BASE AND BASE FOOTPRINT *********************************  -->
+  <!-- Inertial -->
+  <xacro:include filename="$(find bigfootbot_description)/urdf/inertials.urdf.xacro"/>
+  <!-- ********************** ROBOT BASE AND BASE FOOTPRINT *********************************  -->
   <xacro:macro name="base" params="length width height mass wheel_radius wheel_zoff">
     <!-- Define the center of the main robot chassis projected on the ground -->
@@ -15,6 +17,6 @@
         <origin xyz="${length/2} ${-width/2} ${-height/2}" rpy="0 0 1.57079632679"/>
         <geometry>
-          <!--box size="${length} ${width} ${height}"/-->
-          <mesh filename="package://bigfootbot_description/meshes/frame_with_covers_2_m.stl" scale="1.0 1.0 1.0"/> <!-- scale="0.001 0.001 0.001"-->
+          <box size="${length} ${width} ${height}"/>
+          <!--mesh filename="package://bigfootbot_description/meshes/frame_with_covers_2_m.stl" scale="1.0 1.0 1.0"/--> <!-- scale="0.001 0.001 0.001"-->
           <!--mesh filename="file://$(find bigfootbot_description)/meshes/frame_with_covers_2_m.stl" scale="1.0 1.0 1.0"/--> <!-- scale="0.001 0.001 0.001"-->
           <!-- file:// is used instead on package:// because URDF->SDF converter converts package:// to model:// and Gazebo can't fint STLs -->

File: bigfootbot_description/urdf/mech/wheel.urdf.xacro (robot description, xacro)
@@ -1,5 +1,7 @@
 <?xml version="1.0"?>
 <robot xmlns:xacro="http://ros.org/wiki/xacro">
-<!-- *********************** DRIVE WHEELS ******************************  -->
+  <!-- Inertial -->
+  <xacro:include filename="$(find bigfootbot_description)/urdf/inertials.urdf.xacro"/>
+  <!-- *********************** DRIVE WHEELS ******************************  -->
   <xacro:macro name="wheel" params="prefix x_reflect y_reflect rotate_yaw">
     <link name="${prefix}_link">
@@ -7,7 +9,7 @@
         <origin xyz="0 0 0" rpy="0 0 ${rotate_yaw}"/>
         <geometry>
-            <!--cylinder radius="${wheel_radius}" length="${wheel_width}"/-->
+            <cylinder radius="${wheel_radius}" length="${wheel_width}"/>
             <!--mesh filename="package://bigfootbot_description/meshes/wheel.stl" scale="0.001 0.001 0.001"/-->
-            <mesh filename="file://$(find bigfootbot_description)/meshes/wheel.stl" scale="0.001 0.001 0.001"/>
+            <!--mesh filename="file://$(find bigfootbot_description)/meshes/wheel.stl" scale="0.001 0.001 0.001"/-->
             <!-- file:// is used instead on package:// because URDF->SDF converter converts package:// to model:// and Gazebo can't fint STLs -->
         </geometry>
