Commit message: URDF model update, Dockerfiles

File: bigfootbot_description/urdf/inertials.urdf.xacro (robot description, xacro)
@@ -1,5 +1,16 @@
 <?xml version="1.0"?>
 <robot xmlns:xacro="http://ros.org/wiki/xacro">
+  <!--
+  This file defines three macros for calculating the inertial properties of different shapes (box, cylinder, and sphere)
+  used in robot models. The macros return an "inertial" element with the calculated mass and moment of inerti
+  Moment of inertia is a physical quantity that describes how difficult it is to change the rotational
+  motion of an object about an axis. It is a measure of an object's resistance to changes in its rotation rate.
+  The moment of inertia depends on the mass distribution of the object and the axis of rotation.
+  The greater the moment of inertia, the more force is required to change the object's rotation.
+  -->
   <!-- Define intertial property macros  -->
+  <!-- This macro calculates the inertial properties of a box with the given mass, width, height, and depth.
+  The macro uses the parallel axis theorem to calculate the moment of inertia about the center of mass
+  The macro returns an "inertial" element with the calculated mass and moment of inertia. -->
   <xacro:macro name="box_inertia" params="m w h d">
     <inertial>
@@ -9,4 +20,6 @@
     </inertial>
   </xacro:macro>
+  <!-- Calculates the inertial properties of a cylinder with the given mass, radius, and height.
+  The macro returns an "inertial" element with the calculated mass and moment of inertia. -->
   <xacro:macro name="cylinder_inertia" params="m r h">
     <inertial>

File: bigfootbot_description/urdf/mech/base.urdf.xacro (robot description, xacro)
@@ -1,4 +1,12 @@
 <?xml version="1.0"?>
 <robot xmlns:xacro="http://ros.org/wiki/xacro">
+  <!--
+    Macro that creates a robot base (chassis) with given dimensions and properties.
+    The base consists of a link named "base_link" that has a visual and collision element, and a joint named "base_joint"
+    that connects the "base_footprint" link to the "base_link" link.
+    The "base_link" link has a box geometry with dimensions defined by the parameters passed to the macro.
+    The macro also calculates the moments of inertia of the box and returns a block of inertial properties.
+    Finally, the code includes a gazebo tag that defines the visual material of the base in Gazebo.
+  -->
   <!-- Inertial -->
   <xacro:include filename="$(find bigfootbot_description)/urdf/inertials.urdf.xacro"/>
@@ -16,8 +24,9 @@
     <link name="base_link">
       <visual>
-        <origin xyz="${length/2} ${-width/2} ${-height/2}" rpy="0 0 1.57079632679"/>
+        <origin xyz="${length/2} ${-width/2} ${-height/2}" rpy="0 0 1.57079632679"/> <!-- use this origin when <mesh> used as geometry -->
+        <!--origin xyz="0 0 0" rpy="0 0 0"/--> <!-- use this origin when <box> used as geometry -->
         <geometry>
-          <box size="${length} ${width} ${height}"/>
-          <!--mesh filename="package://bigfootbot_description/meshes/frame_with_covers_2_m.stl" scale="1.0 1.0 1.0"/--> <!-- scale="0.001 0.001 0.001"-->
+          <!--box size="${length} ${width} ${height}"/-->
+          <mesh filename="package://bigfootbot_description/meshes/frame_with_covers_2_m.stl" scale="1.0 1.0 1.0"/> <!-- scale="0.001 0.001 0.001"-->
           <!--mesh filename="file://$(find bigfootbot_description)/meshes/frame_with_covers_2_m.stl" scale="1.0 1.0 1.0"/--> <!-- scale="0.001 0.001 0.001"-->
           <!-- file:// is used instead on package:// because URDF->SDF converter converts package:// to model:// and Gazebo can't find STLs
@@ -31,4 +40,6 @@
         </geometry>
       </collision>
+      <!-- Calculates moments of inertia of a box with the given mass, width, length and height and
+      returns block <inertial>...</inertial> -->
       <xacro:box_inertia m="${mass}" w="${width}" d="${length}" h="${height}"/>
     </link>

File: bigfootbot_description/urdf/mech/wheel.urdf.xacro (robot description, xacro)
@@ -1,4 +1,17 @@
 <?xml version="1.0"?>
 <robot xmlns:xacro="http://ros.org/wiki/xacro">
+  <!--
+    Macro that generates a wheel link, collision, and joint for a robot model.
+    The macro takes four parameters: prefix, x_reflect, y_reflect, and rotate_yaw.
+    The prefix parameter is used to name the link and joint. The x_reflect and y_reflect parameters are used to
+    mirror the wheel along the x and y axes, respectively. The rotate_yaw parameter is used to rotate the wheel about the z-axis.
+    The generated wheel link has a cylinder shape with a specified radius and length. It also has a visual and collision element,
+    each with their own origin, geometry, and material properties.
+    The generated joint is a continuous joint that connects the wheel link to the base_link of the robot model.
+    The joint has an axis of rotation along the y-axis and an origin that is offset from the base_link by a specified distance
+    in the x, y, and z directions.
+    The generated wheel link and joint are also configured for use in the Gazebo simulator, with specified friction
+    coefficients and material properties.
+  -->
   <!-- Inertial -->
   <xacro:include filename="$(find bigfootbot_description)/urdf/inertials.urdf.xacro"/>
@@ -9,6 +22,6 @@
         <origin xyz="0 0 0" rpy="0 0 ${rotate_yaw}"/>
         <geometry>
-            <cylinder radius="${wheel_radius}" length="${wheel_width}"/>
-            <!--mesh filename="package://bigfootbot_description/meshes/wheel.stl" scale="0.001 0.001 0.001"/-->
+            <!--cylinder radius="${wheel_radius}" length="${wheel_width}"/-->
+            <mesh filename="package://bigfootbot_description/meshes/wheel.stl" scale="0.001 0.001 0.001"/>
             <!--mesh filename="file://$(find bigfootbot_description)/meshes/wheel.stl" scale="0.001 0.001 0.001"/-->
             <!-- file:// is used instead on package:// because URDF->SDF converter converts package:// to model:// and Gazebo can't fint STLs -->
@@ -53,5 +66,5 @@
       <origin xyz="${x_reflect*wheel_xoff} ${y_reflect*(base_width/2+wheel_ygap)} ${-wheel_zoff}" rpy="0 0 0"/>
       <!--limit upper="3.1415" lower="-3.1415" effort="30" velocity="5.0"/-->
-      <axis xyz="0 1 0"/>
+      <axis xyz="0 1 0"/> <!-- axis of rotation along the y-axis, 1 is the direction of the axis of rotation  -->
     </joint>
   </xacro:macro>
