Commit message: updates

File: basic_mobile_robot/models/basic_mobile_bot_v2.urdf (robot description, URDF)
Before this commit: robot bigfootbot, 4 links, 3 joints
Links:
- added link front_caster; collision sphere radius=${(wheel_radius+wheel_zoff-(base_height/2))}; visual sphere radius=${(wheel_radius+wheel_zoff-(base_height/2))}
- added link gps_link
- link base_link: geometry collision box size=${base_length} ${base_width} ${base_height}; visual mesh filename=package://basic_mobile_robot/meshes/robot_base.stl
Joints:
- added joint caster_joint: type fixed, parent base_link, child front_caster, origin xyz=${caster_xoff} 0.0 ${-(base_height/2)} rpy=0 0 0
- added joint gps_joint: type fixed, parent base_link, child gps_link, origin xyz=0.10 0 0.05 rpy=0 0 0
