Commit message: added xacro files for BarrelBot

File: bigfootbot_description/urdf/mech/wheel.urdf.xacro (robot description, xacro)
@@ -32,5 +32,5 @@
       </visual>
       <collision>
-        <origin xyz="0 0 0" rpy="${pi/2} 0 0"/>
+        <origin xyz="0 0 0" rpy="${pi/2} 0 0"/> <!-- pi/2 = 90 degrees or 1.57 radians (1 radian = 57.2958 degrees) -->
         <geometry>
           <cylinder radius="${wheel_radius}" length="${wheel_width}"/>
