Commit message: docker-compose.yml, base.urdf.xacro

File: bigfootbot_description/urdf/mech/base.urdf.xacro (robot description, xacro)
@@ -16,6 +16,6 @@
         <geometry>
           <!--box size="${length} ${width} ${height}"/-->
-          <!--mesh filename="package://bigfootbot_description/meshes/frame_with_covers_2_m.stl" scale="1.0 1.0 1.0"/--> <!-- scale="0.001 0.001 0.001"-->
-          <mesh filename="file://$(find bigfootbot_description)/meshes/frame_with_covers_2_m.stl" scale="1.0 1.0 1.0"/> <!-- scale="0.001 0.001 0.001"-->
+          <mesh filename="package://bigfootbot_description/meshes/frame_with_covers_2_m.stl" scale="1.0 1.0 1.0"/> <!-- scale="0.001 0.001 0.001"-->
+          <!--mesh filename="file://$(find bigfootbot_description)/meshes/frame_with_covers_2_m.stl" scale="1.0 1.0 1.0"/--> <!-- scale="0.001 0.001 0.001"-->
           <!-- file:// is used instead on package:// because URDF->SDF converter converts package:// to model:// and Gazebo can't fint STLs -->
         </geometry>

Commit message: base.urdf.xacro

File: bigfootbot_description/urdf/mech/base.urdf.xacro (robot description, xacro)
@@ -20,5 +20,5 @@
       <parent link="base_footprint"/>
       <child link="base_link" />
-      <origin xyz="0.0 0.0 ${(wheel_radius+wheel_zoff)}" rpy="0 0 0"/>
+      <origin xyz="0.0 0.0 ${(wheel_radius+wheel_zoff)}" rpy="0 0 0"/> <!-- origin means the position of the child link relative to the parent link -->
     </joint>
     <link name="base_link">

Commit message: updated xacro files, gazebo launch file and rviz launch

File: bigfootbot_description/urdf/mech/base.urdf.xacro (robot description, xacro)
@@ -28,7 +28,8 @@
         <geometry>
           <!--box size="${length} ${width} ${height}"/-->
-          <mesh filename="package://bigfootbot_description/meshes/frame_with_covers_2_m.stl" scale="1.0 1.0 1.0"/> <!-- scale="0.001 0.001 0.001"-->
-          <!--mesh filename="file://$(find bigfootbot_description)/meshes/frame_with_covers_2_m.stl" scale="1.0 1.0 1.0"/--> <!-- scale="0.001 0.001 0.001"-->
+          <!--mesh filename="package://bigfootbot_description/meshes/frame_with_covers_2_m.stl" scale="1.0 1.0 1.0"/--> <!-- scale="0.001 0.001 0.001"-->
+          <mesh filename="file://$(find bigfootbot_description)/meshes/frame_with_covers_2_m.stl" scale="1.0 1.0 1.0"/> <!-- scale="0.001 0.001 0.001"-->
           <!-- file:// is used instead on package:// because URDF->SDF converter converts package:// to model:// and Gazebo can't find STLs -->
+          <!-- RViz can handle both file:// and package:// -->
           <!-- added 03.09.2024: check https://gazebosim.org/docs/harmonic/ros_gz_project_template_guide/#accessing-simulation-assets -->
         </geometry>

File: bigfootbot_description/urdf/mech/wheel.urdf.xacro (robot description, xacro)
@@ -23,7 +23,8 @@
         <geometry>
             <!--cylinder radius="${wheel_radius}" length="${wheel_width}"/-->
-            <mesh filename="package://bigfootbot_description/meshes/wheel.stl" scale="0.001 0.001 0.001"/>
-            <!--mesh filename="file://$(find bigfootbot_description)/meshes/wheel.stl" scale="0.001 0.001 0.001"/-->
+            <!--mesh filename="package://bigfootbot_description/meshes/wheel.stl" scale="0.001 0.001 0.001"/-->
+            <mesh filename="file://$(find bigfootbot_description)/meshes/wheel.stl" scale="0.001 0.001 0.001"/>
             <!-- file:// is used instead on package:// because URDF->SDF converter converts package:// to model:// and Gazebo can't fint STLs -->
+            <!-- RViz can handle both file:// and package:// -->
         </geometry>
         <material name="Gray"> <!-- Material for RViz -->

File: bigfootbot_description/urdf/sensors/imu.urdf.xacro (robot description, xacro)
@@ -8,33 +8,29 @@
       <origin xyz="-0.10 0 0.05" rpy="0 0 0"/>
     </joint>
-    <link name="imu_link"/>
+    <link name="imu_link">
+      <visual>
+        <geometry>
+          <box size="0.05 0.05 0.05"/>
+        </geometry>
+      </visual>
+    </link>
     <!-- *********************** IMU SENSOR SETUP **************************  -->
     <gazebo reference="imu_link">
-      <gravity>true</gravity>
-      <sensor name="bmb_imu" type="imu">
+      <!--gravity>true</gravity-->
+      <sensor name="imu_sensor" type="imu">
+        <!--plugin filename="libgazebo_ros_imu_sensor.so" name="imu_plugin"-->
+        <plugin filename="gz-sim-imu-system"
+                name="gz::sim::systems::Imu">
+          <initial_orientation_as_reference>false</initial_orientation_as_reference>
+          <!--frame_name>imu_link</frame_name-->
+          <ros>
+            <namespace>/demo</namespace>
+            <remapping>~/out:=data</remapping>
+          </ros>
+        </plugin>
         <always_on>true</always_on>
         <update_rate>100</update_rate>
         <visualize>true</visualize>
-        <!--imu>
-          <orientation>
-            <x>
-              <noise type="gaussian">
-                <mean>0.0</mean>
-                <stddev>2e-3</stddev>
-              </noise>
-            </x>
-            <y>
-              <noise type="gaussian">
-                <mean>0.0</mean>
-                <stddev>2e-3</stddev>
-              </noise>
-            </y>
-            <z>
-              <noise type="gaussian">
-                <mean>0.0</mean>
-                <stddev>2e-3</stddev>
-              </noise>
-            </z>
-          </orientation>
+        <imu>
           <angular_velocity>
             <x>
@@ -42,4 +38,6 @@
                 <mean>0.0</mean>
                 <stddev>2e-4</stddev>
+                <bias_mean>0.0000075</bias_mean>
+                <bias_stddev>0.0000008</bias_stddev>
               </noise>
             </x>
@@ -48,4 +46,6 @@
                 <mean>0.0</mean>
                 <stddev>2e-4</stddev>
+                <bias_mean>0.0000075</bias_mean>
+                <bias_stddev>0.0000008</bias_stddev>
               </noise>
             </y>
@@ -54,4 +54,6 @@
                 <mean>0.0</mean>
                 <stddev>2e-4</stddev>
+                <bias_mean>0.0000075</bias_mean>
+                <bias_stddev>0.0000008</bias_stddev>
               </noise>
             </z>
@@ -62,4 +64,6 @@
                 <mean>0.0</mean>
                 <stddev>1.7e-2</stddev>
+                <bias_mean>0.1</bias_mean>
+                <bias_stddev>0.001</bias_stddev>
               </noise>
             </x>
@@ -68,4 +72,6 @@
                 <mean>0.0</mean>
                 <stddev>1.7e-2</stddev>
+                <bias_mean>0.1</bias_mean>
+                <bias_stddev>0.001</bias_stddev>
               </noise>
             </y>
@@ -74,16 +80,10 @@
                 <mean>0.0</mean>
                 <stddev>1.7e-2</stddev>
+                <bias_mean>0.1</bias_mean>
+                <bias_stddev>0.001</bias_stddev>
               </noise>
             </z>
           </linear_acceleration>
-        </imu-->
-        <plugin name="basic_mobile_bot_imu" filename="libgazebo_ros_imu_sensor.so">
-          <initial_orientation_as_reference>false</initial_orientation_as_reference>
-          <frame_name>imu_link</frame_name>
-          <ros>
-            <namespace>/imu</namespace>
-            <remapping>~/out:=data</remapping>
-          </ros>
-        </plugin>
+        </imu>
       </sensor>
     </gazebo>
