Commit message: docker-compose_gazebo.yml teleop->jazzy

File: bigfootbot_description/urdf/sensors/camera.urdf.xacro (robot description, xacro)
@@ -12,5 +12,5 @@
             <box size="0.010 0.03 0.03"/>
         </geometry>
-        <material name="green"/>
+        <material name="Green"/>
       </visual>
       <visual>
@@ -19,5 +19,5 @@
           <cylinder radius="0.002" length="0.1"/>
         </geometry>
-        <material name="green"/>
+        <material name="Green"/>
       </visual>
     </link>
